Commit message: fix: fix tm5 urdf: d6, stl for gazebo

File: tm5_description/urdf/tm5_700.urdf.xacro (robot description, xacro)
@@ -12,5 +12,5 @@
     </inertial>
   </xacro:macro>
-  <xacro:macro name="tm5_700_robot" params="prefix joint_limited
+  <xacro:macro name="tm5_700_robot" params="prefix joint_limited stl_mesh
     shoulder_1_lower_limit:=${-1.5*pi}    shoulder_1_upper_limit:=${1.5*pi}
     shoulder_2_lower_limit:=${-pi}    shoulder_2_upper_limit:=${pi}
@@ -47,5 +47,5 @@
     <xacro:property name="tm_d4" value="0.1222" />
     <xacro:property name="tm_d5" value="0.1060" />
-    <xacro:property name="tm_d6" value="0.1144" />
+    <xacro:property name="tm_d6" value="0.11315" />
     <!-- offsets for shoulder/elbow joints -->
     <xacro:property name="wrist_offset" value="${tm_d5}" />
@@ -70,5 +70,10 @@
       <visual>
         <geometry>
-	      <mesh filename="package://tm5_description/meshes/tm5_900/visual/tm5_base.obj" />
+        <xacro:unless value="${stl_mesh}">
+          <mesh filename="package://tm5_description/meshes/tm5_900/visual/tm5_base.obj" />
+        </xacro:unless>
+        <xacro:if value="${stl_mesh}">
+          <mesh filename="package://tm5_description/meshes/tm5_900/visual/tm5_base.stl" />
+        </xacro:if>
         </geometry>
         <material name="LightGrey">
@@ -78,5 +83,5 @@
       <collision>
         <geometry>
-	      <mesh filename="package://tm5_description/meshes/tm5_900/collision/tm5_base_c.STL" />
+          <mesh filename="package://tm5_description/meshes/tm5_900/collision/tm5_base_c.STL" />
         </geometry>
       </collision>
@@ -99,13 +104,18 @@
       <visual>
         <geometry>
-	      <mesh filename="package://tm5_description/meshes/tm5_900/visual/tm_400w_01.obj" />
-        </geometry>
-        <material name="DarkOlive">
-          <color rgba="0.3 0.3 0.25 1.0" />
-        </material>
-      </visual>
-      <collision>
-        <geometry>
-	      <mesh filename="package://tm5_description/meshes/tm5_900/collision/tm_400w_01_c.STL" />
+        <xacro:unless value="${stl_mesh}">
+          <mesh filename="package://tm5_description/meshes/tm5_900/visual/tm_400w_01.obj" />
+        </xacro:unless>
+        <xacro:if value="${stl_mesh}">
+          <mesh filename="package://tm5_description/meshes/tm5_900/visual/tm_400w_01.stl" />
+        </xacro:if>
+        </geometry>
+        <material name="DarkOlive">
+          <color rgba="0.3 0.3 0.25 1.0" />
+        </material>
+      </visual>
+      <collision>
+        <geometry>
+          <mesh filename="package://tm5_description/meshes/tm5_900/collision/tm_400w_01_c.STL" />
         </geometry>
       </collision>
@@ -128,13 +138,18 @@
       <visual>
         <geometry>
-	      <mesh filename="package://tm5_description/meshes/tm5_700/visual/tm5_700_arm1.obj" />
-        </geometry>
-        <material name="DarkOlive">
-          <color rgba="0.3 0.3 0.25 1.0" />
-        </material>
-      </visual>
-      <collision>
-        <geometry>
-	      <mesh filename="package://tm5_description/meshes/tm5_700/collision/tm5_700_arm1_c.STL" />
+        <xacro:unless value="${stl_mesh}">
+          <mesh filename="package://tm5_description/meshes/tm5_700/visual/tm5_700_arm1.obj" />
+        </xacro:unless>
+        <xacro:if value="${stl_mesh}">
+          <mesh filename="package://tm5_description/meshes/tm5_700/visual/tm5_700_arm1.stl" />
+        </xacro:if>
+        </geometry>
+        <material name="DarkOlive">
+          <color rgba="0.3 0.3 0.25 1.0" />
+        </material>
+      </visual>
+      <collision>
+        <geometry>
+          <mesh filename="package://tm5_description/meshes/tm5_700/collision/tm5_700_arm1_c.STL" />
         </geometry>
       </collision>
@@ -157,13 +172,18 @@
       <visual>
         <geometry>
-	      <mesh filename="package://tm5_description/meshes/tm5_700/visual/tm5_700_arm2.obj" />
-        </geometry>
-        <material name="DarkOlive">
-          <color rgba="0.3 0.3 0.25 1.0" />
-        </material>
-      </visual>
-      <collision>
-        <geometry>
-	  <mesh filename="package://tm5_description/meshes/tm5_700/collision/tm5_700_arm2_c.STL" />
+        <xacro:unless value="${stl_mesh}">
+          <mesh filename="package://tm5_description/meshes/tm5_700/visual/tm5_700_arm2.obj" />
+        </xacro:unless>
+        <xacro:if value="${stl_mesh}">
+          <mesh filename="package://tm5_description/meshes/tm5_700/visual/tm5_700_arm2.stl" />
+        </xacro:if>
+        </geometry>
+        <material name="DarkOlive">
+          <color rgba="0.3 0.3 0.25 1.0" />
+        </material>
+      </visual>
+      <collision>
+        <geometry>
+          <mesh filename="package://tm5_description/meshes/tm5_700/collision/tm5_700_arm2_c.STL" />
         </geometry>
       </collision>
@@ -186,13 +206,18 @@
       <visual>
         <geometry>
-	      <mesh filename="package://tm5_description/meshes/tm5_900/visual/tm_100w_01.obj" />
-        </geometry>
-        <material name="DarkOlive">
-          <color rgba="0.3 0.3 0.25 1.0" />
-        </material>
-      </visual>
-      <collision>
-        <geometry>
-	  <mesh filename="package://tm5_description/meshes/tm5_900/collision/tm_100w_01_c.STL" />
+        <xacro:unless value="${stl_mesh}">
+          <mesh filename="package://tm5_description/meshes/tm5_900/visual/tm_100w_01.obj" />
+        </xacro:unless>
+        <xacro:if value="${stl_mesh}">
+          <mesh filename="package://tm5_description/meshes/tm5_900/visual/tm_100w_01.stl" />
+        </xacro:if>
+        </geometry>
+        <material name="DarkOlive">
+          <color rgba="0.3 0.3 0.25 1.0" />
+        </material>
+      </visual>
+      <collision>
+        <geometry>
+          <mesh filename="package://tm5_description/meshes/tm5_900/collision/tm_100w_01_c.STL" />
         </geometry>
       </collision>
@@ -215,13 +240,18 @@
       <visual>
         <geometry>
-	      <mesh filename="package://tm5_description/meshes/tm5_900/visual/tm_100w_02.obj" />
-        </geometry>
-        <material name="DarkOlive">
-          <color rgba="0.3 0.3 0.25 1.0" />
-        </material>
-      </visual>
-      <collision>
-        <geometry>
-	      <mesh filename="package://tm5_description/meshes/tm5_900/collision/tm_100w_02_c.stl" />
+        <xacro:unless value="${stl_mesh}">
+          <mesh filename="package://tm5_description/meshes/tm5_900/visual/tm_100w_02.obj" />
+        </xacro:unless>
+        <xacro:if value="${stl_mesh}">
+          <mesh filename="package://tm5_description/meshes/tm5_900/visual/tm_100w_02.stl" />
+        </xacro:if>
+        </geometry>
+        <material name="DarkOlive">
+          <color rgba="0.3 0.3 0.25 1.0" />
+        </material>
+      </visual>
+      <collision>
+        <geometry>
+          <mesh filename="package://tm5_description/meshes/tm5_900/collision/tm_100w_02_c.stl" />
         </geometry>
       </collision>
@@ -244,5 +274,10 @@
       <visual>
         <geometry>
-	      <mesh filename="package://tm5_description/meshes/tm5_900/visual/tm_ee.obj" />
+        <xacro:unless value="${stl_mesh}">
+          <mesh filename="package://tm5_description/meshes/tm5_900/visual/tm_ee.obj" />
+        </xacro:unless>
+        <xacro:if value="${stl_mesh}">
+          <mesh filename="package://tm5_description/meshes/tm5_900/visual/tm_ee.stl" />
+        </xacro:if>
         </geometry>
         <material name="LightGrey">
@@ -252,5 +287,5 @@
       <collision>
         <geometry>
-	      <mesh filename="package://tm5_description/meshes/tm5_900/collision/tm_ee_c.stl" />
+          <mesh filename="package://tm5_description/meshes/tm5_900/collision/tm_ee_c.stl" />
         </geometry>
       </collision>

File: tm5_description/urdf/tm5_700_robot.urdf.xacro (robot description, xacro)
@@ -1,5 +1,5 @@
 <?xml version="1.0"?>
 <robot xmlns:xacro="http://wiki.ros.org/xacro" name="tm5_700" >
-  <xacro:arg name="transmission_hw_interface" default="hardware_interface/PositionJointInterface"/>
+  <!-- xacro:arg name="transmission_hw_interface" default="hardware_interface/PositionJointInterface"/-->
   <!-- common stuff -->
   <xacro:include filename="$(find tm5_description)/urdf/common.gazebo.xacro" />
@@ -7,4 +7,11 @@
   <xacro:include filename="$(find tm5_description)/urdf/tm5_700.urdf.xacro" />
   <!-- arm -->
-  <xacro:tm5_700_robot prefix="" joint_limited="false" transmission_hw_interface="$(arg transmission_hw_interface)" />
+  <!--xacro:tm5_700_robot prefix="" joint_limited="false" transmission_hw_interface="$(arg transmission_hw_interface)" /-->
+  <xacro:tm5_700_robot prefix="" joint_limited="false" stl_mesh="$(arg stl_mesh)" />
+  <link name="world" />
+  <joint name="world_joint" type="fixed">
+    <parent link="world" />
+    <child link="base" />
+    <origin xyz="0 0 0" rpy="0 0 0" />
+  </joint>
 </robot>

File: tm5_description/urdf/tm5_900.urdf.xacro (robot description, xacro)
@@ -13,5 +13,5 @@
     </inertial>
   </xacro:macro>
-  <xacro:macro name="tm5_900_robot" params="prefix joint_limited
+  <xacro:macro name="tm5_900_robot" params="prefix joint_limited stl_mesh
     shoulder_1_lower_limit:=${-1.5*pi}    shoulder_1_upper_limit:=${1.5*pi}
     shoulder_2_lower_limit:=${-pi}    shoulder_2_upper_limit:=${pi}
@@ -48,5 +48,5 @@
     <xacro:property name="tm_d4" value="0.1222" />
     <xacro:property name="tm_d5" value="0.1060" />
-    <xacro:property name="tm_d6" value="0.1144" />
+    <xacro:property name="tm_d6" value="0.11315" />
     <!-- offsets for shoulder/elbow joints -->
     <xacro:property name="wrist_offset" value="${tm_d5}" />
@@ -71,5 +71,10 @@
       <visual>
         <geometry>
-	      <mesh filename="package://tm5_description/meshes/tm5_900/visual/tm5_base.obj" />
+        <xacro:unless value="${stl_mesh}">
+          <mesh filename="package://tm5_description/meshes/tm5_900/visual/tm5_base.obj" />
+        </xacro:unless>
+        <xacro:if value="${stl_mesh}">
+          <mesh filename="package://tm5_description/meshes/tm5_900/visual/tm5_base.stl" />
+        </xacro:if>
         </geometry>
         <material name="LightGrey">
@@ -79,5 +84,5 @@
       <collision>
         <geometry>
-	      <mesh filename="package://tm5_description/meshes/tm5_900/collision/tm5_base_c.STL" />
+          <mesh filename="package://tm5_description/meshes/tm5_900/collision/tm5_base_c.STL" />
         </geometry>
       </collision>
@@ -100,13 +105,18 @@
       <visual>
         <geometry>
-	      <mesh filename="package://tm5_description/meshes/tm5_900/visual/tm_400w_01.obj" />
-        </geometry>
-        <material name="DarkOlive">
-          <color rgba="0.3 0.3 0.25 1.0" />
-        </material>
-      </visual>
-      <collision>
-        <geometry>
-	      <mesh filename="package://tm5_description/meshes/tm5_900/collision/tm_400w_01_c.STL" />
+        <xacro:unless value="${stl_mesh}">
+          <mesh filename="package://tm5_description/meshes/tm5_900/visual/tm_400w_01.obj" />
+        </xacro:unless>
+        <xacro:if value="${stl_mesh}">
+          <mesh filename="package://tm5_description/meshes/tm5_900/visual/tm_400w_01.stl" />
+        </xacro:if>
+        </geometry>
+        <material name="DarkOlive">
+          <color rgba="0.3 0.3 0.25 1.0" />
+        </material>
+      </visual>
+      <collision>
+        <geometry>
+          <mesh filename="package://tm5_description/meshes/tm5_900/collision/tm_400w_01_c.STL" />
         </geometry>
       </collision>
@@ -129,13 +139,18 @@
       <visual>
         <geometry>
-	      <mesh filename="package://tm5_description/meshes/tm5_900/visual/tm5_900_arm1.obj" />
-        </geometry>
-        <material name="DarkOlive">
-          <color rgba="0.3 0.3 0.25 1.0" />
-        </material>
-      </visual>
-      <collision>
-        <geometry>
-	      <mesh filename="package://tm5_description/meshes/tm5_900/collision/tm5_900_arm1_c.STL" />
+        <xacro:unless value="${stl_mesh}">
+          <mesh filename="package://tm5_description/meshes/tm5_900/visual/tm5_900_arm1.obj" />
+        </xacro:unless>
+        <xacro:if value="${stl_mesh}">
+          <mesh filename="package://tm5_description/meshes/tm5_900/visual/tm5_900_arm1.stl" />
+        </xacro:if>
+        </geometry>
+        <material name="DarkOlive">
+          <color rgba="0.3 0.3 0.25 1.0" />
+        </material>
+      </visual>
+      <collision>
+        <geometry>
+          <mesh filename="package://tm5_description/meshes/tm5_900/collision/tm5_900_arm1_c.STL" />
         </geometry>
       </collision>
@@ -158,13 +173,18 @@
       <visual>
         <geometry>
-	      <mesh filename="package://tm5_description/meshes/tm5_900/visual/tm5_900_arm2.obj" />
-        </geometry>
-        <material name="DarkOlive">
-          <color rgba="0.3 0.3 0.25 1.0" />
-        </material>
-      </visual>
-      <collision>
-        <geometry>
-	      <mesh filename="package://tm5_description/meshes/tm5_900/collision/tm5_900_arm2_c.STL" />
+        <xacro:unless value="${stl_mesh}">
+          <mesh filename="package://tm5_description/meshes/tm5_900/visual/tm5_900_arm2.obj" />
+        </xacro:unless>
+        <xacro:if value="${stl_mesh}">
+          <mesh filename="package://tm5_description/meshes/tm5_900/visual/tm5_900_arm2.stl" />
+        </xacro:if>
+        </geometry>
+        <material name="DarkOlive">
+          <color rgba="0.3 0.3 0.25 1.0" />
+        </material>
+      </visual>
+      <collision>
+        <geometry>
+          <mesh filename="package://tm5_description/meshes/tm5_900/collision/tm5_900_arm2_c.STL" />
         </geometry>
       </collision>
@@ -187,13 +207,18 @@
       <visual>
         <geometry>
-	      <mesh filename="package://tm5_description/meshes/tm5_900/visual/tm_100w_01.obj" />
-        </geometry>
-        <material name="DarkOlive">
-          <color rgba="0.3 0.3 0.25 1.0" />
-        </material>
-      </visual>
-      <collision>
-        <geometry>
-	      <mesh filename="package://tm5_description/meshes/tm5_900/collision/tm_100w_01_c.STL" />
+        <xacro:unless value="${stl_mesh}">
+          <mesh filename="package://tm5_description/meshes/tm5_900/visual/tm_100w_01.obj" />
+        </xacro:unless>
+        <xacro:if value="${stl_mesh}">
+          <mesh filename="package://tm5_description/meshes/tm5_900/visual/tm_100w_01.stl" />
+        </xacro:if>
+        </geometry>
+        <material name="DarkOlive">
+          <color rgba="0.3 0.3 0.25 1.0" />
+        </material>
+      </visual>
+      <collision>
+        <geometry>
+          <mesh filename="package://tm5_description/meshes/tm5_900/collision/tm_100w_01_c.STL" />
         </geometry>
       </collision>
@@ -216,13 +241,18 @@
       <visual>
         <geometry>
-	      <mesh filename="package://tm5_description/meshes/tm5_900/visual/tm_100w_02.obj" />
-        </geometry>
-        <material name="DarkOlive">
-          <color rgba="0.3 0.3 0.25 1.0" />
-        </material>
-      </visual>
-      <collision>
-        <geometry>
-	      <mesh filename="package://tm5_description/meshes/tm5_900/collision/tm_100w_02_c.stl" />
+        <xacro:unless value="${stl_mesh}">
+          <mesh filename="package://tm5_description/meshes/tm5_900/visual/tm_100w_02.obj" />
+        </xacro:unless>
+        <xacro:if value="${stl_mesh}">
+          <mesh filename="package://tm5_description/meshes/tm5_900/visual/tm_100w_02.stl" />
+        </xacro:if>
+        </geometry>
+        <material name="DarkOlive">
+          <color rgba="0.3 0.3 0.25 1.0" />
+        </material>
+      </visual>
+      <collision>
+        <geometry>
+          <mesh filename="package://tm5_description/meshes/tm5_900/collision/tm_100w_02_c.stl" />
         </geometry>
       </collision>
@@ -245,5 +275,10 @@
       <visual>
         <geometry>
-	      <mesh filename="package://tm5_description/meshes/tm5_900/visual/tm_ee.obj" />
+        <xacro:unless value="${stl_mesh}">
+          <mesh filename="package://tm5_description/meshes/tm5_900/visual/tm_ee.obj" />
+        </xacro:unless>
+        <xacro:if value="${stl_mesh}">
+          <mesh filename="package://tm5_description/meshes/tm5_900/visual/tm_ee.stl" />
+        </xacro:if>
         </geometry>
         <material name="LightGrey">
@@ -253,5 +288,5 @@
       <collision>
         <geometry>
-	      <mesh filename="package://tm5_description/meshes/tm5_900/collision/tm_ee_c.stl" />
+          <mesh filename="package://tm5_description/meshes/tm5_900/collision/tm_ee_c.stl" />
         </geometry>
       </collision>

File: tm5_description/urdf/tm5_900_robot.urdf.xacro (robot description, xacro)
@@ -8,4 +8,10 @@
   <!-- arm -->
   <!--xacro:tm5_900_robot prefix="" joint_limited="false" transmission_hw_interface="$(arg transmission_hw_interface)" /-->
-  <xacro:tm5_900_robot prefix="" joint_limited="false"/>
+  <xacro:tm5_900_robot prefix="" joint_limited="false" stl_mesh="$(arg stl_mesh)" />
+  <link name="world" />
+  <joint name="world_joint" type="fixed">
+    <parent link="world" />
+    <child link="base" />
+    <origin xyz="0 0 0" rpy="0 0 0" />
+  </joint>
 </robot>

Commit message: fix: fix tm5 DH parameters

File: tm5_description/urdf/tm5_700.urdf.xacro (robot description, xacro)
@@ -35,5 +35,5 @@
       DH for TM5-700:
       a = [0.0000, 0.3290, 0.3115,  0.0000,  0.0000,  0.0000]
-      d = [0.1452,  0.0000,  0.0000,  -0.1222,  0.1060,  0.1144]
+      d = [0.1452,  0.0000,  0.0000,  -0.1223,  0.1060,  0.11315]
       alpha = [-0.5*pi, 0, 0, 0.5*pi, 0.5*pi, 0]
       q_home_offset = [0, -0.5*pi, 0, 0.5*pi, 0, 0]
@@ -45,5 +45,5 @@
     <xacro:property name="tm_a2" value="0.3290" />
     <xacro:property name="tm_a3" value="0.3115" />
-    <xacro:property name="tm_d4" value="0.1222" />
+    <xacro:property name="tm_d4" value="0.1223" />
     <xacro:property name="tm_d5" value="0.1060" />
     <xacro:property name="tm_d6" value="0.11315" />
@@ -51,5 +51,5 @@
     <xacro:property name="wrist_offset" value="${tm_d5}" />
     <xacro:property name="shoulder_offset" value="0.146" />
-    <xacro:property name="elbow_offset" value="${wrist_offset + shoulder_offset - tm_d4}" /> <!-- 0.1298 -->
+    <xacro:property name="elbow_offset" value="${wrist_offset + shoulder_offset - tm_d4}" /> <!-- 0.1297 -->
     <!-- link lengths -->
     <xacro:property name="shoulder_height" value="${tm_d1}" />

File: tm5_description/urdf/tm5_900.urdf.xacro (robot description, xacro)
@@ -36,5 +36,5 @@
       DH for TM5-900:
       a = [0.0000, 0.4290, 0.4115,  0.0000,  0.0000,  0.0000]
-      d = [0.1452,  0.0000,  0.0000,  -0.1222,  0.1060,  0.1144]
+      d = [0.1452,  0.0000,  0.0000,  -0.1223,  0.1060,  0.11315]
       alpha = [-0.5*pi, 0, 0, 0.5*pi, 0.5*pi, 0]
       q_home_offset = [0, -0.5*pi, 0, 0.5*pi, 0, 0]
@@ -46,5 +46,5 @@
     <xacro:property name="tm_a2" value="0.4290" />
     <xacro:property name="tm_a3" value="0.4115" />
-    <xacro:property name="tm_d4" value="0.1222" />
+    <xacro:property name="tm_d4" value="0.1223" />
     <xacro:property name="tm_d5" value="0.1060" />
     <xacro:property name="tm_d6" value="0.11315" />
@@ -52,5 +52,5 @@
     <xacro:property name="wrist_offset" value="${tm_d5}" />
     <xacro:property name="shoulder_offset" value="0.146" />
-    <xacro:property name="elbow_offset" value="${wrist_offset + shoulder_offset - tm_d4}" /> <!-- 0.1298 -->
+    <xacro:property name="elbow_offset" value="${wrist_offset + shoulder_offset - tm_d4}" /> <!-- 0.1297 -->
     <!-- link lengths -->
     <xacro:property name="shoulder_height" value="${tm_d1}" />

File: tm5_description/urdf/tm5_900_simple.urdf (robot description, URDF)
Before this commit: robot tm5_900, 9 links, 8 joints
Joints:
- joint elbow_joint: origin xyz=0 0.429 -0.1298 rpy=0 0 0 -> xyz=0 0.429 -0.1297 rpy=0 0 0
- joint wrist_3_joint: origin xyz=0 0 0.1144 rpy=0 0 0 -> xyz=0 0 0.11315 rpy=0 0 0
