Commit message: fix: gazebo can't open .obj, using .stl for now

File: tm12_description/urdf/tm12.urdf.xacro (robot description, xacro)
@@ -12,5 +12,5 @@
     </inertial>
   </xacro:macro>
-  <xacro:macro name="tm12_robot" params="prefix joint_limited
+  <xacro:macro name="tm12_robot" params="prefix joint_limited stl_mesh
     shoulder_1_lower_limit:=${-1.5*pi}    shoulder_1_upper_limit:=${1.5*pi}
     shoulder_2_lower_limit:=${-pi}    shoulder_2_upper_limit:=${pi}
@@ -70,5 +70,10 @@
       <visual>
         <geometry>
-	      <mesh filename="package://tm12_description/meshes/tm12_1300/visual/tm12_base.obj" />
+        <xacro:unless value="${stl_mesh}">
+          <mesh filename="package://tm12_description/meshes/tm12_1300/visual/tm12_base.obj" />
+        </xacro:unless>
+        <xacro:if value="${stl_mesh}">
+          <mesh filename="package://tm12_description/meshes/tm12_1300/visual/tm12_base.stl" />
+        </xacro:if>
         </geometry>
         <material name="LightGrey">
@@ -78,5 +83,5 @@
       <collision>
         <geometry>
-	      <mesh filename="package://tm12_description/meshes/tm12_1300/collision/tm12_base_c.STL" />
+          <mesh filename="package://tm12_description/meshes/tm12_1300/collision/tm12_base_c.STL" />
         </geometry>
       </collision>
@@ -99,13 +104,18 @@
       <visual>
         <geometry>
-	      <mesh filename="package://tm12_description/meshes/tm12_1300/visual/tm_750w_01.obj" />
-        </geometry>
-        <material name="DarkOlive">
-          <color rgba="0.3 0.3 0.25 1.0" />
-        </material>
-      </visual>
-      <collision>
-        <geometry>
-	      <mesh filename="package://tm12_description/meshes/tm12_1300/collision/tm_750w_01_c.STL" />
+        <xacro:unless value="${stl_mesh}">
+          <mesh filename="package://tm12_description/meshes/tm12_1300/visual/tm_750w_01.obj" />
+        </xacro:unless>
+        <xacro:if value="${stl_mesh}">
+          <mesh filename="package://tm12_description/meshes/tm12_1300/visual/tm_750w_01.stl" />
+        </xacro:if>
+        </geometry>
+        <material name="DarkOlive">
+          <color rgba="0.3 0.3 0.25 1.0" />
+        </material>
+      </visual>
+      <collision>
+        <geometry>
+          <mesh filename="package://tm12_description/meshes/tm12_1300/collision/tm_750w_01_c.STL" />
         </geometry>
       </collision>
@@ -128,13 +138,18 @@
       <visual>
         <geometry>
-	      <mesh filename="package://tm12_description/meshes/tm12_1300/visual/tm12_arm1.obj" />
-        </geometry>
-        <material name="DarkOlive">
-          <color rgba="0.3 0.3 0.25 1.0" />
-        </material>
-      </visual>
-      <collision>
-        <geometry>
-	      <mesh filename="package://tm12_description/meshes/tm12_1300/collision/tm12_arm1_c.STL" />
+        <xacro:unless value="${stl_mesh}">
+          <mesh filename="package://tm12_description/meshes/tm12_1300/visual/tm12_arm1.obj" />
+        </xacro:unless>
+        <xacro:if value="${stl_mesh}">
+          <mesh filename="package://tm12_description/meshes/tm12_1300/visual/tm12_arm1.stl" />
+        </xacro:if>
+        </geometry>
+        <material name="DarkOlive">
+          <color rgba="0.3 0.3 0.25 1.0" />
+        </material>
+      </visual>
+      <collision>
+        <geometry>
+          <mesh filename="package://tm12_description/meshes/tm12_1300/collision/tm12_arm1_c.STL" />
         </geometry>
       </collision>
@@ -157,13 +172,18 @@
       <visual>
         <geometry>
-	      <mesh filename="package://tm12_description/meshes/tm12_1300/visual/tm12_arm2.obj" />
-        </geometry>
-        <material name="DarkOlive">
-          <color rgba="0.3 0.3 0.25 1.0" />
-        </material>
-      </visual>
-      <collision>
-        <geometry>
-	      <mesh filename="package://tm12_description/meshes/tm12_1300/collision/tm12_arm2_c.STL" />
+        <xacro:unless value="${stl_mesh}">
+          <mesh filename="package://tm12_description/meshes/tm12_1300/visual/tm12_arm2.obj" />
+        </xacro:unless>
+        <xacro:if value="${stl_mesh}">
+          <mesh filename="package://tm12_description/meshes/tm12_1300/visual/tm12_arm2.stl" />
+        </xacro:if>
+        </geometry>
+        <material name="DarkOlive">
+          <color rgba="0.3 0.3 0.25 1.0" />
+        </material>
+      </visual>
+      <collision>
+        <geometry>
+          <mesh filename="package://tm12_description/meshes/tm12_1300/collision/tm12_arm2_c.STL" />
         </geometry>
       </collision>
@@ -186,13 +206,18 @@
       <visual>
         <geometry>
-	      <mesh filename="package://tm12_description/meshes/tm12_1300/visual/tm_100w_01.obj" />
-        </geometry>
-        <material name="DarkOlive">
-          <color rgba="0.3 0.3 0.25 1.0" />
-        </material>
-      </visual>
-      <collision>
-        <geometry>
-	      <mesh filename="package://tm12_description/meshes/tm12_1300/collision/tm_100w_01_c.STL" />
+        <xacro:unless value="${stl_mesh}">
+          <mesh filename="package://tm12_description/meshes/tm12_1300/visual/tm_100w_01.obj" />
+        </xacro:unless>
+        <xacro:if value="${stl_mesh}">
+          <mesh filename="package://tm12_description/meshes/tm12_1300/visual/tm_100w_01.stl" />
+        </xacro:if>
+        </geometry>
+        <material name="DarkOlive">
+          <color rgba="0.3 0.3 0.25 1.0" />
+        </material>
+      </visual>
+      <collision>
+        <geometry>
+          <mesh filename="package://tm12_description/meshes/tm12_1300/collision/tm_100w_01_c.STL" />
         </geometry>
       </collision>
@@ -215,13 +240,18 @@
       <visual>
         <geometry>
-	      <mesh filename="package://tm12_description/meshes/tm12_1300/visual/tm_100w_02.obj" />
-        </geometry>
-        <material name="DarkOlive">
-          <color rgba="0.3 0.3 0.25 1.0" />
-        </material>
-      </visual>
-      <collision>
-        <geometry>
-	      <mesh filename="package://tm12_description/meshes/tm12_1300/collision/tm_100w_02_c.stl" />
+        <xacro:unless value="${stl_mesh}">
+          <mesh filename="package://tm12_description/meshes/tm12_1300/visual/tm_100w_02.obj" />
+        </xacro:unless>
+        <xacro:if value="${stl_mesh}">
+          <mesh filename="package://tm12_description/meshes/tm12_1300/visual/tm_100w_02.stl" />
+        </xacro:if>
+        </geometry>
+        <material name="DarkOlive">
+          <color rgba="0.3 0.3 0.25 1.0" />
+        </material>
+      </visual>
+      <collision>
+        <geometry>
+          <mesh filename="package://tm12_description/meshes/tm12_1300/collision/tm_100w_02_c.stl" />
         </geometry>
       </collision>
@@ -244,5 +274,10 @@
       <visual>
         <geometry>
-	      <mesh filename="package://tm12_description/meshes/tm12_1300/visual/tm_ee.obj" />
+        <xacro:unless value="${stl_mesh}">
+          <mesh filename="package://tm12_description/meshes/tm12_1300/visual/tm_ee.obj" />
+        </xacro:unless>
+        <xacro:if value="${stl_mesh}">
+          <mesh filename="package://tm12_description/meshes/tm12_1300/visual/tm_ee.stl" />
+        </xacro:if>
         </geometry>
         <material name="LightGrey">
@@ -252,5 +287,5 @@
       <collision>
         <geometry>
-	      <mesh filename="package://tm12_description/meshes/tm12_1300/collision/tm_ee_c.stl" />
+          <mesh filename="package://tm12_description/meshes/tm12_1300/collision/tm_ee_c.stl" />
         </geometry>
       </collision>

File: tm12_description/urdf/tm12_robot.urdf.xacro (robot description, xacro)
@@ -1,5 +1,5 @@
 <?xml version="1.0"?>
 <robot xmlns:xacro="http://wiki.ros.org/xacro" name="tm12" >
-  <xacro:arg name="transmission_hw_interface" default="hardware_interface/PositionJointInterface"/>
+  <!--xacro:arg name="transmission_hw_interface" default="hardware_interface/PositionJointInterface"/-->
   <!-- common stuff -->
   <xacro:include filename="$(find tm5_description)/urdf/common.gazebo.xacro" />
@@ -7,4 +7,11 @@
   <xacro:include filename="$(find tm12_description)/urdf/tm12.urdf.xacro" />
   <!-- arm -->
-  <xacro:tm12_robot prefix="" joint_limited="false" transmission_hw_interface="$(arg transmission_hw_interface)" />
+  <!--xacro:tm12_robot prefix="" joint_limited="false" transmission_hw_interface="$(arg transmission_hw_interface)" /-->
+  <xacro:tm12_robot prefix="" joint_limited="false" stl_mesh="$(arg stl_mesh)" />
+  <link name="world" />
+  <joint name="world_joint" type="fixed">
+    <parent link="world" />
+    <child link="base" />
+    <origin xyz="0 0 0" rpy="0 0 0" />
+  </joint>
 </robot>

Commit message: fix link inertial parameters

File: tm12_description/urdf/tm12.urdf.xacro (robot description, xacro)
@@ -3,5 +3,14 @@
   <xacro:include filename="$(find tm5_description)/urdf/tm.transmission.xacro" />
   <xacro:include filename="$(find tm5_description)/urdf/tm.gazebo.xacro" />
-  <xacro:macro name="cylinder_inertial" params="radius length mass *origin">
+  <xacro:macro name="cylinder_inertial_y" params="radius length mass *origin">
+    <inertial>
+      <mass value="${mass}" />
+      <xacro:insert_block name="origin" />
+      <inertia ixx="${0.0833333 * mass * (3 * radius * radius + length * length)}" ixy="0.0" ixz="0.0"
+        iyy="${0.5 * mass * radius * radius}" iyz="0.0"
+        izz="${0.0833333 * mass * (3 * radius * radius + length * length)}" />
+    </inertial>
+  </xacro:macro>
+  <xacro:macro name="cylinder_inertial_z" params="radius length mass *origin">
     <inertial>
       <mass value="${mass}" />
@@ -86,7 +95,7 @@
         </geometry>
       </collision>
-      <xacro:cylinder_inertial radius="0.06" length="0.05" mass="${base_mass}">
-        <origin xyz="0 0 0" rpy="0 0 0" />
-      </xacro:cylinder_inertial>
+      <xacro:cylinder_inertial_y radius="0.06" length="0.05" mass="${base_mass}">
+        <origin xyz="0 0 0" rpy="0 0 0" />
+      </xacro:cylinder_inertial_y>
     </link>
     <joint name="${prefix}shoulder_1_joint" type="revolute">
@@ -120,7 +129,7 @@
         </geometry>
       </collision>
-      <xacro:cylinder_inertial radius="0.06" length="0.15" mass="${shoulder_mass}">
-        <origin xyz="0 0 0" rpy="0 0 0" />
-      </xacro:cylinder_inertial>
+      <xacro:cylinder_inertial_y radius="0.06" length="0.15" mass="${shoulder_mass}">
+        <origin xyz="0 0 0" rpy="0 0 0" />
+      </xacro:cylinder_inertial_y>
     </link>
     <joint name="${prefix}shoulder_2_joint" type="revolute">
@@ -154,7 +163,7 @@
         </geometry>
       </collision>
-      <xacro:cylinder_inertial radius="0.06" length="${arm_1_length}" mass="${arm_1_mass}">
-        <origin xyz="0 0 ${0.5*arm_1_length}" rpy="0 0 0" />
-      </xacro:cylinder_inertial>
+      <xacro:cylinder_inertial_y radius="0.06" length="${arm_1_length}" mass="${arm_1_mass}">
+        <origin xyz="0 ${0.5*arm_1_length} 0" rpy="0 0 0" />
+      </xacro:cylinder_inertial_y>
     </link>
     <joint name="${prefix}elbow_joint" type="revolute">
@@ -188,7 +197,7 @@
         </geometry>
       </collision>
-      <xacro:cylinder_inertial radius="0.045" length="${arm_2_length}" mass="${arm_2_mass}">
-        <origin xyz="0 0 ${0.5*arm_2_length}" rpy="0 0 0" />
-      </xacro:cylinder_inertial>
+      <xacro:cylinder_inertial_y radius="0.045" length="${arm_2_length}" mass="${arm_2_mass}">
+        <origin xyz="0 ${0.5*arm_2_length} 0" rpy="0 0 0" />
+      </xacro:cylinder_inertial_y>
     </link>
     <joint name="${prefix}wrist_1_joint" type="revolute">
@@ -222,7 +231,7 @@
         </geometry>
       </collision>
-      <xacro:cylinder_inertial radius="0.045" length="0.12" mass="${wrist_1_mass}">
-        <origin xyz="0 0 0" rpy="0 0 0" />
-      </xacro:cylinder_inertial>
+      <xacro:cylinder_inertial_y radius="0.045" length="0.12" mass="${wrist_1_mass}">
+        <origin xyz="0 0 0" rpy="0 0 0" />
+      </xacro:cylinder_inertial_y>
     </link>
     <joint name="${prefix}wrist_2_joint" type="revolute">
@@ -256,7 +265,7 @@
         </geometry>
       </collision>
-      <xacro:cylinder_inertial radius="0.045" length="0.12" mass="${wrist_2_mass}">
-        <origin xyz="0 0 0" rpy="0 0 0" />
-      </xacro:cylinder_inertial>
+      <xacro:cylinder_inertial_z radius="0.045" length="0.12" mass="${wrist_2_mass}">
+        <origin xyz="0 0 0" rpy="0 0 0" />
+      </xacro:cylinder_inertial_z>
     </link>
     <joint name="${prefix}wrist_3_joint" type="revolute">
@@ -290,7 +299,7 @@
         </geometry>
       </collision>
-      <xacro:cylinder_inertial radius="0.045" length="0.12" mass="${wrist_3_mass}">
-        <origin xyz="0 0 0" rpy="0 0 0" />
-      </xacro:cylinder_inertial>
+      <xacro:cylinder_inertial_z radius="0.045" length="0.06" mass="${wrist_3_mass}">
+        <origin xyz="0 0 0" rpy="0 0 0" />
+      </xacro:cylinder_inertial_z>
     </link>
     <joint name="${prefix}flange_fixed_joint" type="fixed">

File: tm5_description/urdf/tm5_700.urdf.xacro (robot description, xacro)
@@ -3,5 +3,14 @@
   <xacro:include filename="$(find tm5_description)/urdf/tm.transmission.xacro" />
   <xacro:include filename="$(find tm5_description)/urdf/tm.gazebo.xacro" />
-  <xacro:macro name="cylinder_inertial" params="radius length mass *origin">
+  <xacro:macro name="cylinder_inertial_y" params="radius length mass *origin">
+    <inertial>
+      <mass value="${mass}" />
+      <xacro:insert_block name="origin" />
+      <inertia ixx="${0.0833333 * mass * (3 * radius * radius + length * length)}" ixy="0.0" ixz="0.0"
+        iyy="${0.5 * mass * radius * radius}" iyz="0.0"
+        izz="${0.0833333 * mass * (3 * radius * radius + length * length)}" />
+    </inertial>
+  </xacro:macro>
+  <xacro:macro name="cylinder_inertial_z" params="radius length mass *origin">
     <inertial>
       <mass value="${mass}" />
@@ -86,7 +95,7 @@
         </geometry>
       </collision>
-      <xacro:cylinder_inertial radius="0.06" length="0.05" mass="${base_mass}">
-        <origin xyz="0 0 0" rpy="0 0 0" />
-      </xacro:cylinder_inertial>
+      <xacro:cylinder_inertial_y radius="0.06" length="0.05" mass="${base_mass}">
+        <origin xyz="0 0 0" rpy="0 0 0" />
+      </xacro:cylinder_inertial_y>
     </link>
     <joint name="${prefix}shoulder_1_joint" type="revolute">
@@ -120,7 +129,7 @@
         </geometry>
       </collision>
-      <xacro:cylinder_inertial radius="0.06" length="0.15" mass="${shoulder_mass}">
-        <origin xyz="0 0 0" rpy="0 0 0" />
-      </xacro:cylinder_inertial>
+      <xacro:cylinder_inertial_y radius="0.06" length="0.15" mass="${shoulder_mass}">
+        <origin xyz="0 0 0" rpy="0 0 0" />
+      </xacro:cylinder_inertial_y>
     </link>
     <joint name="${prefix}shoulder_2_joint" type="revolute">
@@ -154,7 +163,7 @@
         </geometry>
       </collision>
-      <xacro:cylinder_inertial radius="0.06" length="${arm_1_length}" mass="${arm_1_mass}">
-        <origin xyz="0 0 ${0.5*arm_1_length}" rpy="0 0 0" />
-      </xacro:cylinder_inertial>
+      <xacro:cylinder_inertial_y radius="0.06" length="${arm_1_length}" mass="${arm_1_mass}">
+        <origin xyz="0 ${0.5*arm_1_length} 0" rpy="0 0 0" />
+      </xacro:cylinder_inertial_y>
     </link>
     <joint name="${prefix}elbow_joint" type="revolute">
@@ -188,7 +197,7 @@
         </geometry>
       </collision>
-      <xacro:cylinder_inertial radius="0.045" length="${arm_2_length}" mass="${arm_2_mass}">
-        <origin xyz="0 0 ${0.5*arm_2_length}" rpy="0 0 0" />
-      </xacro:cylinder_inertial>
+      <xacro:cylinder_inertial_y radius="0.045" length="${arm_2_length}" mass="${arm_2_mass}">
+        <origin xyz="0 ${0.5*arm_2_length} 0" rpy="0 0 0" />
+      </xacro:cylinder_inertial_y>
     </link>
     <joint name="${prefix}wrist_1_joint" type="revolute">
@@ -222,7 +231,7 @@
         </geometry>
       </collision>
-      <xacro:cylinder_inertial radius="0.045" length="0.12" mass="${wrist_1_mass}">
-        <origin xyz="0 0 0" rpy="0 0 0" />
-      </xacro:cylinder_inertial>
+      <xacro:cylinder_inertial_y radius="0.045" length="0.06" mass="${wrist_1_mass}">
+        <origin xyz="0 0 0" rpy="0 0 0" />
+      </xacro:cylinder_inertial_y>
     </link>
     <joint name="${prefix}wrist_2_joint" type="revolute">
@@ -256,7 +265,7 @@
         </geometry>
       </collision>
-      <xacro:cylinder_inertial radius="0.045" length="0.12" mass="${wrist_2_mass}">
-        <origin xyz="0 0 0" rpy="0 0 0" />
-      </xacro:cylinder_inertial>
+      <xacro:cylinder_inertial_z radius="0.045" length="0.12" mass="${wrist_2_mass}">
+        <origin xyz="0 0 0" rpy="0 0 0" />
+      </xacro:cylinder_inertial_z>
     </link>
     <joint name="${prefix}wrist_3_joint" type="revolute">
@@ -290,7 +299,7 @@
         </geometry>
       </collision>
-      <xacro:cylinder_inertial radius="0.045" length="0.12" mass="${wrist_3_mass}">
-        <origin xyz="0 0 0" rpy="0 0 0" />
-      </xacro:cylinder_inertial>
+      <xacro:cylinder_inertial_z radius="0.045" length="0.12" mass="${wrist_3_mass}">
+        <origin xyz="0 0 0" rpy="0 0 0" />
+      </xacro:cylinder_inertial_z>
     </link>
     <joint name="${prefix}flange_fixed_joint" type="fixed">

File: tm5_description/urdf/tm5_700_robot.urdf.xacro (robot description, xacro)
@@ -2,4 +2,5 @@
 <robot xmlns:xacro="http://wiki.ros.org/xacro" name="tm5_700" >
   <!-- xacro:arg name="transmission_hw_interface" default="hardware_interface/PositionJointInterface"/-->
+  <xacro:arg name="stl_mesh" default="false"/>
   <!-- common stuff -->
   <xacro:include filename="$(find tm5_description)/urdf/common.gazebo.xacro" />

File: tm5_description/urdf/tm5_900.urdf.xacro (robot description, xacro)
@@ -4,5 +4,14 @@
   <xacro:include filename="$(find tm5_description)/urdf/tm.transmission.xacro" />
   <!--xacro:include filename="$(find tm5_description)/urdf/tm.gazebo.xacro" /-->
-  <xacro:macro name="cylinder_inertial" params="radius length mass *origin">
+  <xacro:macro name="cylinder_inertial_y" params="radius length mass *origin">
+    <inertial>
+      <mass value="${mass}" />
+      <xacro:insert_block name="origin" />
+      <inertia ixx="${0.0833333 * mass * (3 * radius * radius + length * length)}" ixy="0.0" ixz="0.0"
+        iyy="${0.5 * mass * radius * radius}" iyz="0.0"
+        izz="${0.0833333 * mass * (3 * radius * radius + length * length)}" />
+    </inertial>
+  </xacro:macro>
+  <xacro:macro name="cylinder_inertial_z" params="radius length mass *origin">
     <inertial>
       <mass value="${mass}" />
@@ -87,7 +96,7 @@
         </geometry>
       </collision>
-      <xacro:cylinder_inertial radius="0.06" length="0.05" mass="${base_mass}">
-        <origin xyz="0 0 0" rpy="0 0 0" />
-      </xacro:cylinder_inertial>
+      <xacro:cylinder_inertial_y radius="0.06" length="0.05" mass="${base_mass}">
+        <origin xyz="0 0 0" rpy="0 0 0" />
+      </xacro:cylinder_inertial_y>
     </link>
     <joint name="${prefix}shoulder_1_joint" type="revolute">
@@ -121,7 +130,7 @@
         </geometry>
       </collision>
-      <xacro:cylinder_inertial radius="0.06" length="0.15" mass="${shoulder_mass}">
-        <origin xyz="0 0 0" rpy="0 0 0" />
-      </xacro:cylinder_inertial>
+      <xacro:cylinder_inertial_y radius="0.06" length="0.15" mass="${shoulder_mass}">
+        <origin xyz="0 0 0" rpy="0 0 0" />
+      </xacro:cylinder_inertial_y>
     </link>
     <joint name="${prefix}shoulder_2_joint" type="revolute">
@@ -155,7 +164,7 @@
         </geometry>
       </collision>
-      <xacro:cylinder_inertial radius="0.06" length="${arm_1_length}" mass="${arm_1_mass}">
-        <origin xyz="0 0 ${0.5*arm_1_length}" rpy="0 0 0" />
-      </xacro:cylinder_inertial>
+      <xacro:cylinder_inertial_y radius="0.06" length="${arm_1_length}" mass="${arm_1_mass}">
+        <origin xyz="0 ${0.5*arm_1_length} 0" rpy="0 0 0" />
+      </xacro:cylinder_inertial_y>
     </link>
     <joint name="${prefix}elbow_joint" type="revolute">
@@ -189,7 +198,7 @@
         </geometry>
       </collision>
-      <xacro:cylinder_inertial radius="0.045" length="${arm_2_length}" mass="${arm_2_mass}">
-        <origin xyz="0 0 ${0.5*arm_2_length}" rpy="0 0 0" />
-      </xacro:cylinder_inertial>
+      <xacro:cylinder_inertial_y radius="0.045" length="${arm_2_length}" mass="${arm_2_mass}">
+        <origin xyz="0 ${0.5*arm_2_length} 0" rpy="0 0 0" />
+      </xacro:cylinder_inertial_y>
     </link>
     <joint name="${prefix}wrist_1_joint" type="revolute">
@@ -223,7 +232,7 @@
         </geometry>
       </collision>
-      <xacro:cylinder_inertial radius="0.045" length="0.12" mass="${wrist_1_mass}">
-        <origin xyz="0 0 0" rpy="0 0 0" />
-      </xacro:cylinder_inertial>
+      <xacro:cylinder_inertial_y radius="0.045" length="0.12" mass="${wrist_1_mass}">
+        <origin xyz="0 0 0" rpy="0 0 0" />
+      </xacro:cylinder_inertial_y>
     </link>
     <joint name="${prefix}wrist_2_joint" type="revolute">
@@ -257,7 +266,7 @@
         </geometry>
       </collision>
-      <xacro:cylinder_inertial radius="0.045" length="0.12" mass="${wrist_2_mass}">
-        <origin xyz="0 0 0" rpy="0 0 0" />
-      </xacro:cylinder_inertial>
+      <xacro:cylinder_inertial_z radius="0.045" length="0.12" mass="${wrist_2_mass}">
+        <origin xyz="0 0 0" rpy="0 0 0" />
+      </xacro:cylinder_inertial_z>
     </link>
     <joint name="${prefix}wrist_3_joint" type="revolute">
@@ -291,7 +300,7 @@
         </geometry>
       </collision>
-      <xacro:cylinder_inertial radius="0.045" length="0.12" mass="${wrist_3_mass}">
-        <origin xyz="0 0 0" rpy="0 0 0" />
-      </xacro:cylinder_inertial>
+      <xacro:cylinder_inertial_z radius="0.045" length="0.06" mass="${wrist_3_mass}">
+        <origin xyz="0 0 0" rpy="0 0 0" />
+      </xacro:cylinder_inertial_z>
     </link>
     <joint name="${prefix}flange_fixed_joint" type="fixed">

File: tm5_description/urdf/tm5_900_robot.urdf.xacro (robot description, xacro)
@@ -2,4 +2,5 @@
 <robot xmlns:xacro="http://wiki.ros.org/xacro" name="tm5_900" >
   <!--xacro:arg name="transmission_hw_interface" default="hardware_interface/PositionJointInterface"/-->
+  <!--xacro:arg name="stl_mesh" default="false"/-->
   <!-- common stuff -->
   <xacro:include filename="$(find tm5_description)/urdf/common.gazebo.xacro" />
