Commit message: 1.5.9 modify *.STL to *.stl of meshes files, some URDF and launch files and update README.md.

File: tm12_description/urdf/tm12.urdf.xacro (robot description, xacro)
@@ -92,5 +92,5 @@
       <collision>
         <geometry>
-          <mesh filename="package://tm12_description/meshes/tm12_1300/collision/tm12_base_c.STL" />
+          <mesh filename="package://tm12_description/meshes/tm12_1300/collision/tm12_base_c.stl" />
         </geometry>
       </collision>
@@ -126,5 +126,5 @@
       <collision>
         <geometry>
-          <mesh filename="package://tm12_description/meshes/tm12_1300/collision/tm_750w_01_c.STL" />
+          <mesh filename="package://tm12_description/meshes/tm12_1300/collision/tm_750w_01_c.stl" />
         </geometry>
       </collision>
@@ -160,5 +160,5 @@
       <collision>
         <geometry>
-          <mesh filename="package://tm12_description/meshes/tm12_1300/collision/tm12_arm1_c.STL" />
+          <mesh filename="package://tm12_description/meshes/tm12_1300/collision/tm12_arm1_c.stl" />
         </geometry>
       </collision>
@@ -194,5 +194,5 @@
       <collision>
         <geometry>
-          <mesh filename="package://tm12_description/meshes/tm12_1300/collision/tm12_arm2_c.STL" />
+          <mesh filename="package://tm12_description/meshes/tm12_1300/collision/tm12_arm2_c.stl" />
         </geometry>
       </collision>
@@ -228,5 +228,5 @@
       <collision>
         <geometry>
-          <mesh filename="package://tm12_description/meshes/tm12_1300/collision/tm_100w_01_c.STL" />
+          <mesh filename="package://tm12_description/meshes/tm12_1300/collision/tm_100w_01_c.stl" />
         </geometry>
       </collision>

File: tm5_description/urdf/tm5_700.urdf.xacro (robot description, xacro)
@@ -92,5 +92,5 @@
       <collision>
         <geometry>
-          <mesh filename="package://tm5_description/meshes/tm5_900/collision/tm5_base_c.STL" />
+          <mesh filename="package://tm5_description/meshes/tm5_900/collision/tm5_base_c.stl" />
         </geometry>
       </collision>
@@ -126,5 +126,5 @@
       <collision>
         <geometry>
-          <mesh filename="package://tm5_description/meshes/tm5_900/collision/tm_400w_01_c.STL" />
+          <mesh filename="package://tm5_description/meshes/tm5_900/collision/tm_400w_01_c.stl" />
         </geometry>
       </collision>
@@ -160,5 +160,5 @@
       <collision>
         <geometry>
-          <mesh filename="package://tm5_description/meshes/tm5_700/collision/tm5_700_arm1_c.STL" />
+          <mesh filename="package://tm5_description/meshes/tm5_700/collision/tm5_700_arm1_c.stl" />
         </geometry>
       </collision>
@@ -194,5 +194,5 @@
       <collision>
         <geometry>
-          <mesh filename="package://tm5_description/meshes/tm5_700/collision/tm5_700_arm2_c.STL" />
+          <mesh filename="package://tm5_description/meshes/tm5_700/collision/tm5_700_arm2_c.stl" />
         </geometry>
       </collision>
@@ -228,5 +228,5 @@
       <collision>
         <geometry>
-          <mesh filename="package://tm5_description/meshes/tm5_900/collision/tm_100w_01_c.STL" />
+          <mesh filename="package://tm5_description/meshes/tm5_900/collision/tm_100w_01_c.stl" />
         </geometry>
       </collision>

File: tm5_description/urdf/tm5_900.urdf.xacro (robot description, xacro)
@@ -93,5 +93,5 @@
       <collision>
         <geometry>
-          <mesh filename="package://tm5_description/meshes/tm5_900/collision/tm5_base_c.STL" />
+          <mesh filename="package://tm5_description/meshes/tm5_900/collision/tm5_base_c.stl" />
         </geometry>
       </collision>
@@ -127,5 +127,5 @@
       <collision>
         <geometry>
-          <mesh filename="package://tm5_description/meshes/tm5_900/collision/tm_400w_01_c.STL" />
+          <mesh filename="package://tm5_description/meshes/tm5_900/collision/tm_400w_01_c.stl" />
         </geometry>
       </collision>
@@ -161,5 +161,5 @@
       <collision>
         <geometry>
-          <mesh filename="package://tm5_description/meshes/tm5_900/collision/tm5_900_arm1_c.STL" />
+          <mesh filename="package://tm5_description/meshes/tm5_900/collision/tm5_900_arm1_c.stl" />
         </geometry>
       </collision>
@@ -195,5 +195,5 @@
       <collision>
         <geometry>
-          <mesh filename="package://tm5_description/meshes/tm5_900/collision/tm5_900_arm2_c.STL" />
+          <mesh filename="package://tm5_description/meshes/tm5_900/collision/tm5_900_arm2_c.stl" />
         </geometry>
       </collision>
@@ -229,5 +229,5 @@
       <collision>
         <geometry>
-          <mesh filename="package://tm5_description/meshes/tm5_900/collision/tm_100w_01_c.STL" />
+          <mesh filename="package://tm5_description/meshes/tm5_900/collision/tm_100w_01_c.stl" />
         </geometry>
       </collision>
