Commit message: 1.9.9 modify the joint range value of J1,J2,J4,J5,J6 of the eyeless urdf,xacro models and update README.md.

File: tm_description/urdf/tm12x-nominal.urdf (robot description, URDF)
Before this commit: robot tm12x, 11 links, 10 joints
Joints:
- joint shoulder_1_joint: limit lower=-4.71238898038469 upper=4.71238898038469 effort=353 velocity=2.0943951023931953 -> lower=-6.283185307179586 upper=6.283185307179586 effort=353 velocity=2.0943951023931953
- joint shoulder_2_joint: limit lower=-3.141592653589793 upper=3.141592653589793 effort=353 velocity=2.0943951023931953 -> lower=-6.283185307179586 upper=6.283185307179586 effort=353 velocity=2.0943951023931953
- joint wrist_1_joint: limit lower=-3.141592653589793 upper=3.141592653589793 effort=54 velocity=3.141592653589793 -> lower=-6.283185307179586 upper=6.283185307179586 effort=54 velocity=3.141592653589793
- joint wrist_2_joint: limit lower=-3.141592653589793 upper=3.141592653589793 effort=54 velocity=3.141592653589793 -> lower=-6.283185307179586 upper=6.283185307179586 effort=54 velocity=3.141592653589793
- joint wrist_3_joint: limit lower=-4.71238898038469 upper=4.71238898038469 effort=54 velocity=3.141592653589793 -> lower=-6.283185307179586 upper=6.283185307179586 effort=54 velocity=3.141592653589793

File: tm_description/urdf/tm14x-nominal.urdf (robot description, URDF)
Before this commit: robot tm14x, 11 links, 10 joints
Joints:
- joint shoulder_1_joint: limit lower=-4.71238898038469 upper=4.71238898038469 effort=353 velocity=2.0943951023931953 -> lower=-6.283185307179586 upper=6.283185307179586 effort=353 velocity=2.0943951023931953
- joint shoulder_2_joint: limit lower=-3.141592653589793 upper=3.141592653589793 effort=353 velocity=2.0943951023931953 -> lower=-6.283185307179586 upper=6.283185307179586 effort=353 velocity=2.0943951023931953
- joint wrist_1_joint: limit lower=-3.141592653589793 upper=3.141592653589793 effort=54 velocity=2.6179938779914944 -> lower=-6.283185307179586 upper=6.283185307179586 effort=54 velocity=2.6179938779914944
- joint wrist_2_joint: limit lower=-3.141592653589793 upper=3.141592653589793 effort=54 velocity=2.6179938779914944 -> lower=-6.283185307179586 upper=6.283185307179586 effort=54 velocity=2.6179938779914944
- joint wrist_3_joint: limit lower=-4.71238898038469 upper=4.71238898038469 effort=54 velocity=3.141592653589793 -> lower=-6.283185307179586 upper=6.283185307179586 effort=54 velocity=3.141592653589793

File: tm_description/urdf/tm5x-700-nominal.urdf (robot description, URDF)
Before this commit: robot tm5x-700, 11 links, 10 joints
Joints:
- joint shoulder_1_joint: limit lower=-4.71238898038469 upper=4.71238898038469 effort=157 velocity=3.141592653589793 -> lower=-6.283185307179586 upper=6.283185307179586 effort=157 velocity=3.141592653589793
- joint shoulder_2_joint: limit lower=-3.141592653589793 upper=3.141592653589793 effort=157 velocity=3.141592653589793 -> lower=-6.283185307179586 upper=6.283185307179586 effort=157 velocity=3.141592653589793
- joint wrist_1_joint: limit lower=-3.141592653589793 upper=3.141592653589793 effort=43 velocity=3.9269908169872414 -> lower=-6.283185307179586 upper=6.283185307179586 effort=43 velocity=3.9269908169872414
- joint wrist_2_joint: limit lower=-3.141592653589793 upper=3.141592653589793 effort=43 velocity=3.9269908169872414 -> lower=-6.283185307179586 upper=6.283185307179586 effort=43 velocity=3.9269908169872414
- joint wrist_3_joint: limit lower=-4.71238898038469 upper=4.71238898038469 effort=43 velocity=3.9269908169872414 -> lower=-6.283185307179586 upper=6.283185307179586 effort=43 velocity=3.9269908169872414

File: tm_description/urdf/tm5x-900-nominal.urdf (robot description, URDF)
Before this commit: robot tm5x-900, 11 links, 10 joints
Joints:
- joint shoulder_1_joint: limit lower=-4.71238898038469 upper=4.71238898038469 effort=157 velocity=3.141592653589793 -> lower=-6.283185307179586 upper=6.283185307179586 effort=157 velocity=3.141592653589793
- joint shoulder_2_joint: limit lower=-3.141592653589793 upper=3.141592653589793 effort=157 velocity=3.141592653589793 -> lower=-6.283185307179586 upper=6.283185307179586 effort=157 velocity=3.141592653589793
- joint wrist_1_joint: limit lower=-3.141592653589793 upper=3.141592653589793 effort=43 velocity=3.9269908169872414 -> lower=-6.283185307179586 upper=6.283185307179586 effort=43 velocity=3.9269908169872414
- joint wrist_2_joint: limit lower=-3.141592653589793 upper=3.141592653589793 effort=43 velocity=3.9269908169872414 -> lower=-6.283185307179586 upper=6.283185307179586 effort=43 velocity=3.9269908169872414
- joint wrist_3_joint: limit lower=-4.71238898038469 upper=4.71238898038469 effort=43 velocity=3.9269908169872414 -> lower=-6.283185307179586 upper=6.283185307179586 effort=43 velocity=3.9269908169872414

File: tm_description/xacro/macro.tm12x-nominal.urdf.xacro (robot description, xacro)
@@ -3,10 +3,10 @@
   <xacro:include filename="$(find tm_description)/xacro/macro.inertial.xacro" />
   <xacro:macro name="tm12x" params="ns prefix color:=none format:=obj
-    shoulder_1_joint_lower_limit:=${radians(-270)}    shoulder_1_joint_upper_limit:=${radians(270)}
-    shoulder_2_joint_lower_limit:=${radians(-180)}    shoulder_2_joint_upper_limit:=${radians(180)}
+    shoulder_1_joint_lower_limit:=${radians(-360)}    shoulder_1_joint_upper_limit:=${radians(360)}
+    shoulder_2_joint_lower_limit:=${radians(-360)}    shoulder_2_joint_upper_limit:=${radians(360)}
     elbow_joint_lower_limit:=${radians(-166)}    elbow_joint_upper_limit:=${radians(166)}
-    wrist_1_joint_lower_limit:=${radians(-180)}    wrist_1_joint_upper_limit:=${radians(180)}
-    wrist_2_joint_lower_limit:=${radians(-180)}    wrist_2_joint_upper_limit:=${radians(180)}
-    wrist_3_joint_lower_limit:=${radians(-270)}    wrist_3_joint_upper_limit:=${radians(270)}
+    wrist_1_joint_lower_limit:=${radians(-360)}    wrist_1_joint_upper_limit:=${radians(360)}
+    wrist_2_joint_lower_limit:=${radians(-360)}    wrist_2_joint_upper_limit:=${radians(360)}
+    wrist_3_joint_lower_limit:=${radians(-360)}    wrist_3_joint_upper_limit:=${radians(360)}
     shoulder_1_joint_velocity_limit:=${radians(120)}
     shoulder_2_joint_velocity_limit:=${radians(120)}

File: tm_description/xacro/macro.tm5x-700-nominal.urdf.xacro (robot description, xacro)
@@ -3,10 +3,10 @@
   <xacro:include filename="$(find tm_description)/xacro/macro.inertial.xacro" />
   <xacro:macro name="tm5x-700" params="ns prefix color:=none format:=obj
-    shoulder_1_joint_lower_limit:=${radians(-270)}    shoulder_1_joint_upper_limit:=${radians(270)}
-    shoulder_2_joint_lower_limit:=${radians(-180)}    shoulder_2_joint_upper_limit:=${radians(180)}
+    shoulder_1_joint_lower_limit:=${radians(-360)}    shoulder_1_joint_upper_limit:=${radians(360)}
+    shoulder_2_joint_lower_limit:=${radians(-360)}    shoulder_2_joint_upper_limit:=${radians(360)}
     elbow_joint_lower_limit:=${radians(-155)}    elbow_joint_upper_limit:=${radians(155)}
-    wrist_1_joint_lower_limit:=${radians(-180)}    wrist_1_joint_upper_limit:=${radians(180)}
-    wrist_2_joint_lower_limit:=${radians(-180)}    wrist_2_joint_upper_limit:=${radians(180)}
-    wrist_3_joint_lower_limit:=${radians(-270)}    wrist_3_joint_upper_limit:=${radians(270)}
+    wrist_1_joint_lower_limit:=${radians(-360)}    wrist_1_joint_upper_limit:=${radians(360)}
+    wrist_2_joint_lower_limit:=${radians(-360)}    wrist_2_joint_upper_limit:=${radians(360)}
+    wrist_3_joint_lower_limit:=${radians(-360)}    wrist_3_joint_upper_limit:=${radians(360)}
     shoulder_1_joint_velocity_limit:=${radians(180)}
     shoulder_2_joint_velocity_limit:=${radians(180)}

File: tm_description/xacro/macro.tm5x-900-nominal.urdf.xacro (robot description, xacro)
@@ -3,10 +3,10 @@
   <xacro:include filename="$(find tm_description)/xacro/macro.inertial.xacro" />
   <xacro:macro name="tm5x-900" params="ns prefix color:=none format:=obj
-    shoulder_1_joint_lower_limit:=${radians(-270)}    shoulder_1_joint_upper_limit:=${radians(270)}
-    shoulder_2_joint_lower_limit:=${radians(-180)}    shoulder_2_joint_upper_limit:=${radians(180)}
+    shoulder_1_joint_lower_limit:=${radians(-360)}    shoulder_1_joint_upper_limit:=${radians(360)}
+    shoulder_2_joint_lower_limit:=${radians(-360)}    shoulder_2_joint_upper_limit:=${radians(360)}
     elbow_joint_lower_limit:=${radians(-155)}    elbow_joint_upper_limit:=${radians(155)}
-    wrist_1_joint_lower_limit:=${radians(-180)}    wrist_1_joint_upper_limit:=${radians(180)}
-    wrist_2_joint_lower_limit:=${radians(-180)}    wrist_2_joint_upper_limit:=${radians(180)}
-    wrist_3_joint_lower_limit:=${radians(-270)}    wrist_3_joint_upper_limit:=${radians(270)}
+    wrist_1_joint_lower_limit:=${radians(-360)}    wrist_1_joint_upper_limit:=${radians(360)}
+    wrist_2_joint_lower_limit:=${radians(-360)}    wrist_2_joint_upper_limit:=${radians(360)}
+    wrist_3_joint_lower_limit:=${radians(-360)}    wrist_3_joint_upper_limit:=${radians(360)}
     shoulder_1_joint_velocity_limit:=${radians(180)}
     shoulder_2_joint_velocity_limit:=${radians(180)}

File: tm_gazebo/urdf/tm12x-nominal.urdf (robot description, URDF)
Before this commit: robot tm12x, 11 links, 10 joints
Joints:
- joint shoulder_1_joint: limit lower=-4.71238898038 upper=4.71238898038 effort=353 velocity=2.09439510239 -> lower=-6.28318530718 upper=6.28318530718 effort=353 velocity=2.09439510239
- joint shoulder_2_joint: limit lower=-3.14159265359 upper=3.14159265359 effort=353 velocity=2.09439510239 -> lower=-6.28318530718 upper=6.28318530718 effort=353 velocity=2.09439510239
- joint wrist_1_joint: limit lower=-3.14159265359 upper=3.14159265359 effort=54 velocity=3.14159265359 -> lower=-6.28318530718 upper=6.28318530718 effort=54 velocity=3.14159265359
- joint wrist_2_joint: limit lower=-3.14159265359 upper=3.14159265359 effort=54 velocity=3.14159265359 -> lower=-6.28318530718 upper=6.28318530718 effort=54 velocity=3.14159265359
- joint wrist_3_joint: limit lower=-4.71238898038 upper=4.71238898038 effort=54 velocity=3.14159265359 -> lower=-6.28318530718 upper=6.28318530718 effort=54 velocity=3.14159265359

File: tm_gazebo/urdf/tm14x-nominal.urdf (robot description, URDF)
Before this commit: robot tm14x, 11 links, 10 joints
Joints:
- joint shoulder_1_joint: limit lower=-4.71238898038 upper=4.71238898038 effort=353 velocity=2.09439510239 -> lower=-6.28318530718 upper=6.28318530718 effort=353 velocity=2.09439510239
- joint shoulder_2_joint: limit lower=-3.14159265359 upper=3.14159265359 effort=353 velocity=2.09439510239 -> lower=-6.28318530718 upper=6.28318530718 effort=353 velocity=2.09439510239
- joint wrist_1_joint: limit lower=-3.14159265359 upper=3.14159265359 effort=54 velocity=2.61799387799 -> lower=-6.28318530718 upper=6.28318530718 effort=54 velocity=2.61799387799
- joint wrist_2_joint: limit lower=-3.14159265359 upper=3.14159265359 effort=54 velocity=2.61799387799 -> lower=-6.28318530718 upper=6.28318530718 effort=54 velocity=2.61799387799
- joint wrist_3_joint: limit lower=-4.71238898038 upper=4.71238898038 effort=54 velocity=3.14159265359 -> lower=-6.28318530718 upper=6.28318530718 effort=54 velocity=3.14159265359

File: tm_gazebo/urdf/tm5x-700-nominal.urdf (robot description, URDF)
Before this commit: robot tm5x-700, 11 links, 10 joints
Joints:
- joint shoulder_1_joint: limit lower=-4.71238898038 upper=4.71238898038 effort=157 velocity=3.14159265359 -> lower=-6.28318530718 upper=6.28318530718 effort=157 velocity=3.14159265359
- joint shoulder_2_joint: limit lower=-3.14159265359 upper=3.14159265359 effort=157 velocity=3.14159265359 -> lower=-6.28318530718 upper=6.28318530718 effort=157 velocity=3.14159265359
- joint wrist_1_joint: limit lower=-3.14159265359 upper=3.14159265359 effort=43 velocity=3.92699081699 -> lower=-6.28318530718 upper=6.28318530718 effort=43 velocity=3.92699081699
- joint wrist_2_joint: limit lower=-3.14159265359 upper=3.14159265359 effort=43 velocity=3.92699081699 -> lower=-6.28318530718 upper=6.28318530718 effort=43 velocity=3.92699081699
- joint wrist_3_joint: limit lower=-4.71238898038 upper=4.71238898038 effort=43 velocity=3.92699081699 -> lower=-6.28318530718 upper=6.28318530718 effort=43 velocity=3.92699081699

File: tm_gazebo/urdf/tm5x-900-nominal.urdf (robot description, URDF)
Before this commit: robot tm5x-900, 11 links, 10 joints
Joints:
- joint shoulder_1_joint: limit lower=-4.71238898038 upper=4.71238898038 effort=157 velocity=3.14159265359 -> lower=-6.28318530718 upper=6.28318530718 effort=157 velocity=3.14159265359
- joint shoulder_2_joint: limit lower=-3.14159265359 upper=3.14159265359 effort=157 velocity=3.14159265359 -> lower=-6.28318530718 upper=6.28318530718 effort=157 velocity=3.14159265359
- joint wrist_1_joint: limit lower=-3.14159265359 upper=3.14159265359 effort=43 velocity=3.92699081699 -> lower=-6.28318530718 upper=6.28318530718 effort=43 velocity=3.92699081699
- joint wrist_2_joint: limit lower=-3.14159265359 upper=3.14159265359 effort=43 velocity=3.92699081699 -> lower=-6.28318530718 upper=6.28318530718 effort=43 velocity=3.92699081699
- joint wrist_3_joint: limit lower=-4.71238898038 upper=4.71238898038 effort=43 velocity=3.92699081699 -> lower=-6.28318530718 upper=6.28318530718 effort=43 velocity=3.92699081699
